File: pcb/_restore_backup_2026-08-18T15-40-20-313/twoporthub.kicad_sch (KiCad schematic)
At the start: 37 parts, among them IC1 TS3USB221ERSER, J1 USB_C_16P, J2 USB_C_16P, J3 USB_C_16P, J4 USB_A, J5 USB_A, J6 USB_C_16P, SW1 SW_Push_DPDT, U1 SL2.1A, U2 TPD4E001DBVR, U3 TPD4E001DBVR, U4 TLV77312PDBVR

Commit message: Added 3.3v regulator
Parts:
- removed C15: 100nF, symbol Device:C
- removed C16: 1uF, symbol Device:C
- removed U3: TPD4E001DBVR, DBV6, symbol Project:TPD4E001DBVR
- removed U4: TLV77312PDBVR, DBV0005A-IPC_A, symbol Project:TLV77312PDBVR
- C9: value 1uF -> 100nF
Connections:
- net +3.3V: now also C13.1, C14.1, U1.13 (VDD3); no longer C8.1, C9.2
- net GND: now also C9.2, R8.2; no longer C9.1, IC1.5 (GND), R8.1
- net IN2_CC1: no longer names the net of J6.A5 (CC1)
- net IN2_CC1: now also R8.1; no longer R8.2
- net IN2_CC2: no longer names the net of J6.B5 (CC2), R7.2
- new net: C8.1, C9.1, IC1.5 (GND)
Other:
- moved on the sheet: C5, IC1, R9, SW1
