File: pcb/_restore_backup_2026-08-18T18-22-39-525/twoporthub.kicad_pcb (KiCad board)
At the start: 2 copper layers, 70 x 74.5 mm, 36 parts, among them IC1 TS3USB221ERSER, J1 USB_A, J2 USB_A, J3 USB_C_16P, J4 USB_C_16P, J5 USB_C_16P, J6 USB_C_16P, SW1 SW_Push_DPDT, U1 SL2.1A, U2 TLV77312PDBVR, U3 TPD4E001DBVR, U4 TPD4E001DBVR

Commit message: Worked until I realized some traces might be impossible
Parts:
- C12: value 100nF -> 1uF
- moved SW1 8.86 mm to (205.5, 71.0)
- moved C4 7.78 mm to (186.7, 69.0)
- moved U2 7.56 mm to (213.2, 84.1)
- moved C11 7.27 mm to (214.0, 87.0), turned to 0 degrees
- moved R5 5.49 mm to (219.0, 73.0), turned to 0 degrees
- moved C12 5.26 mm to (208.3, 76.0), turned to 180 degrees
- moved R3 1.97 mm to (187.0, 70.5), turned to 0 degrees
- moved C13 1.10 mm to (219.1, 78.5)
- moved R1 0.69 mm to (185.3, 80.5)
Connections:
- C12 pad 1: +5V -> BYPASS
- C12 pad 2: BYPASS -> +3.3V
- IC1 pad 1: IN2_D+ -> IN1_D+
- IC1 pad 2: IN2_D- -> IN1_D-
- IC1 pad 3: IN1_D+ -> IN2_D+
- IC1 pad 4: IN1_D- -> IN2_D-
Routing:
- net +5V: track 75.5 -> 0.00 mm
- net D3+: track 16.4 -> 0.00 mm
- net D3-: track 16.1 -> 0.00 mm
- net D1-: track 15.8 -> 0.00 mm
- net D2-: track 14.6 -> 0.00 mm
- net D4-: track 14.4 -> 0.00 mm
- net D4+: track 13.7 -> 0.00 mm
- net BYPASS: track 100.9 -> 87.2 mm, vias 2 -> 0
- net Net-(IC1-S): track 13.1 -> 0.00 mm
- net D2+: track 12.9 -> 0.00 mm
- net +3.3V: track 12.6 -> 0.00 mm
- net D1+: track 12.2 -> 0.00 mm
- net IN2_D-: track 23.3 -> 12.6 mm
- net IN2_D+: track 21.1 -> 10.6 mm
- net IN1_D+: track 23.8 -> 15.5 mm
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- removed copper zone on F.Cu, net BYPASS
